File: kicad/Keypad.sch (KiCad schematic (older format))
At the start: 19 parts

Commit message: just a test
Other:
- note added: "Keypad"
- moved on the sheet: R?
Changed lines of the file:
@@
 Connection ~ 10100 2450
 Wire Wire Line
-	7450 1550 9900 1550
+	7050 1550 9900 1550
 Connection ~ 9400 1550
 Wire Wire Line
-	7450 1900 9900 1900
+	7050 1900 9900 1900
 Connection ~ 9400 1900
 Wire Wire Line
-	7450 2250 9900 2250
+	7050 2250 9900 2250
 Connection ~ 9400 2250
 Wire Wire Line
-	7450 2600 9900 2600
+	7050 2600 9900 2600
 Connection ~ 9400 2600
 Connection ~ 8900 1900
@@
 Connection ~ 8900 1550
 Wire Wire Line
-	7800 4950 9100 4950
+	7400 4950 9100 4950
 Connection ~ 9100 2800
 Wire Wire Line
-	7800 5250 9600 5250
+	7400 5250 9600 5250
 Connection ~ 9600 2800
 Wire Wire Line
-	7800 5550 10100 5550
+	7400 5550 10100 5550
 Connection ~ 10100 2800
 $Comp
 L R R?
 U 1 1 58248CAD
-P 8100 4650
-F 0 "R?" V 8180 4650 50  0000 C CNN
-F 1 "18k" V 8100 4650 50  0000 C CNN
-F 2 "" V 8030 4650 50  0000 C CNN
-F 3 "" H 8100 4650 50  0000 C CNN
-	1    8100 4650
+P 7700 4650
+F 0 "R?" V 7780 4650 50  0000 C CNN
+F 1 "18k" V 7700 4650 50  0000 C CNN
+F 2 "" V 7630 4650 50  0000 C CNN
+F 3 "" H 7700 4650 50  0000 C CNN
+	1    7700 4650
 	1    0    0    -1
 $EndComp
@@
 L R R?
 U 1 1 58248CB4
-P 8400 4650
-F 0 "R?" V 8480 4650 50  0000 C CNN
-F 1 "18k" V 8400 4650 50  0000 C CNN
-F 2 "" V 8330 4650 50  0000 C CNN
-F 3 "" H 8400 4650 50  0000 C CNN
-	1    8400 4650
+P 8000 4650
+F 0 "R?" V 8080 4650 50  0000 C CNN
+F 1 "18k" V 8000 4650 50  0000 C CNN
+F 2 "" V 7930 4650 50  0000 C CNN
+F 3 "" H 8000 4650 50  0000 C CNN
+	1    8000 4650
 	1    0    0    -1
 $EndComp
@@
 L R R?
 U 1 1 58248CBB
-P 8700 4650
-F 0 "R?" V 8780 4650 50  0000 C CNN
-F 1 "18k" V 8700 4650 50  0000 C CNN
-F 2 "" V 8630 4650 50  0000 C CNN
-F 3 "" H 8700 4650 50  0000 C CNN
-	1    8700 4650
+P 8300 4650
+F 0 "R?" V 8380 4650 50  0000 C CNN
+F 1 "18k" V 8300 4650 50  0000 C CNN
+F 2 "" V 8230 4650 50  0000 C CNN
+F 3 "" H 8300 4650 50  0000 C CNN
+	1    8300 4650
 	1    0    0    -1
 $EndComp
 Wire Wire Line
-	8100 4800 8100 4950
-Connection ~ 8100 4950
+	7700 4800 7700 4950
+Connection ~ 7700 4950
 Wire Wire Line
-	8400 4800 8400 5250
-Connection ~ 8400 5250
+	8000 4800 8000 5250
+Connection ~ 8000 5250
 Wire Wire Line
-	8700 4800 8700 5550
-Connection ~ 8700 5550
+	8300 4800 8300 5550
+Connection ~ 8300 5550
 $Comp
 L +3.3V #PWR?
 U 1 1 58248CC8
-P 8700 4100
-F 0 "#PWR?" H 8700 3950 50  0001 C CNN
-F 1 "+3.3V" H 8700 4240 50  0000 C CNN
-F 2 "" H 8700 4100 50  0000 C CNN
-F 3 "" H 8700 4100 50  0000 C CNN
-	1    8700 4100
+P 8300 4100
+F 0 "#PWR?" H 8300 3950 50  0001 C CNN
+F 1 "+3.3V" H 8300 4240 50  0000 C CNN
+F 2 "" H 8300 4100 50  0000 C CNN
+F 3 "" H 8300 4100 50  0000 C CNN
+	1    8300 4100
 	1    0    0    -1
 $EndComp
 Wire Wire Line
-	8700 4100 8700 4500
+	8300 4100 8300 4500
 Wire Wire Line
-	8400 4500 8400 4350
-Connection ~ 8400 4350
+	8000 4500 8000 4350
+Connection ~ 8000 4350
 Wire Wire Line
-	8100 4500 8100 4350
+	7700 4500 7700 4350
 $Comp
 L R R?
 U 1 1 58248CD2
-P 7700 2950
-F 0 "R?" V 7780 2950 50  0000 C CNN
-F 1 "2k2" V 7700 2950 50  0000 C CNN
-F 2 "" V 7630 2950 50  0000 C CNN
-F 3 "" H 7700 2950 50  0000 C CNN
-	1    7700 2950
+P 7300 2950
+F 0 "R?" V 7380 2950 50  0000 C CNN
+F 1 "2k2" V 7300 2950 50  0000 C CNN
+F 2 "" V 7230 2950 50  0000 C CNN
+F 3 "" H 7300 2950 50  0000 C CNN
+	1    7300 2950
 	1    0    0    -1
 $EndComp
@@
 L R R?
 U 1 1 58248CD9
-P 8000 2950
-F 0 "R?" V 8080 2950 50  0000 C CNN
-F 1 "2k2" V 8000 2950 50  0000 C CNN
-F 2 "" V 7930 2950 50  0000 C CNN
-F 3 "" H 8000 2950 50  0000 C CNN
-	1    8000 2950
+P 7600 2950
+F 0 "R?" V 7680 2950 50  0000 C CNN
+F 1 "2k2" V 7600 2950 50  0000 C CNN
+F 2 "" V 7530 2950 50  0000 C CNN
+F 3 "" H 7600 2950 50  0000 C CNN
+	1    7600 2950
 	1    0    0    -1
 $EndComp
@@
 L R R?
 U 1 1 58248CE0
-P 8300 2950
-F 0 "R?" V 8380 2950 50  0000 C CNN
-F 1 "2k2" V 8300 2950 50  0000 C CNN
-F 2 "" V 8230 2950 50  0000 C CNN
-F 3 "" H 8300 2950 50  0000 C CNN
-	1    8300 2950
+P 7900 2950
+F 0 "R?" V 7980 2950 50  0000 C CNN
+F 1 "2k2" V 7900 2950 50  0000 C CNN
+F 2 "" V 7830 2950 50  0000 C CNN
+F 3 "" H 7900 2950 50  0000 C CNN
+	1    7900 2950
 	1    0    0    -1
 $EndComp
 Wire Wire Line
-	7700 3250 8700 3250
-Connection ~ 8000 3250
+	7300 3250 8300 3250
+Connection ~ 7600 3250
 $Comp
 L R R?
 U 1 1 58248CE9
-P 8600 2950
-F 0 "R?" V 8680 2950 50  0000 C CNN
-F 1 "2k2" V 8600 2950 50  0000 C CNN
-F 2 "" V 8530 2950 50  0000 C CNN
-F 3 "" H 8600 2950 50  0000 C CNN
-	1    8600 2950
+P 8200 2950
+F 0 "R?" V 8280 2950 50  0000 C CNN
+F 1 "2k2" V 8200 2950 50  0000 C CNN
+F 2 "" V 8130 2950 50  0000 C CNN
+F 3 "" H 8200 2950 50  0000 C CNN
+	1    8200 2950
 	1    0    0    -1
 $EndComp
-Connection ~ 8600 2600
-Connection ~ 8300 3250
-Connection ~ 8300 2250
-Connection ~ 8000 1900
+Connection ~ 8200 2600
+Connection ~ 7900 3250
+Connection ~ 7900 2250
+Connection ~ 7600 1900
 $Comp
 L GND #PWR?
 U 1 1 58248CF4
-P 8700 3500
-F 0 "#PWR?" H 8700 3250 50  0001 C CNN
-F 1 "GND" H 8700 3350 50  0000 C CNN
-F 2 "" H 8700 3500 50  0000 C CNN
-F 3 "" H 8700 3500 50  0000 C CNN
-	1    8700 3500
+P 8300 3500
+F 0 "#PWR?" H 8300 3250 50  0001 C CNN
+F 1 "GND" H 8300 3350 50  0000 C CNN
+F 2 "" H 8300 3500 50  0000 C CNN
+F 3 "" H 8300 3500 50  0000 C CNN
+	1    8300 3500
 	1    0    0    -1
 $EndComp
-Connection ~ 7700 1550
+Connection ~ 7300 1550
 Wire Wire Line
-	7700 2800 7700 1550
+	7300 2800 7300 1550
 Wire Wire Line
-	8000 2800 8000 1900
+	7600 2800 7600 1900
 Wire Wire Line
-	8300 2800 8300 2250
+	7900 2800 7900 2250
 Wire Wire Line
-	8600 2800 8600 2600
+	8200 2800 8200 2600
 Wire Wire Line
-	8600 3250 8600 3100
+	8200 3250 8200 3100
 Wire Wire Line
-	8300 3100 8300 3250
+	7900 3100 7900 3250
 Wire Wire Line
-	8000 3100 8000 3250
+	7600 3100 7600 3250
 Wire Wire Line
-	7700 3100 7700 3250
+	7300 3100 7300 3250
 Wire Wire Line
-	8700 3250 8700 3500
-Connection ~ 8600 3250
+	8300 3250 8300 3500
+Connection ~ 8200 3250
 Wire Wire Line
-	8100 4350 8700 4350
-Connection ~ 8700 4350
+	7700 4350 8300 4350
+Connection ~ 8300 4350
+Wire Notes Line
+	8700 1350 10300 1350
+Wire Notes Line
+	10300 1350 10300 3050
+Wire Notes Line
+	10300 3050 8700 3050
+Wire Notes Line
+	8700 3050 8700 1350
+Text Notes 8700 1300 0    60   ~ 0
+Keypad
 $EndSCHEMATC
